Commit message: Add Hokuyo transforms to pepper.urdf and pepper_sensors.xacro

File: pepper_description/urdf/pepper1.0_generated_urdf/pepper.urdf (robot description, URDF)
Before this commit: robot JulietteY20MP, 83 links, 82 joints
Links:
- added link HokuyoLaser_frame
Joints:
- added joint LaserSensor/Hokuyo_sensor_fixedjoint: type fixed, parent Tibia, child HokuyoLaser_frame, origin xyz=0.2 0 -0.289 rpy=0 0 0, axis 0 0 0

File: pepper_description/urdf/pepper1.0_generated_urdf/pepper_sensors.xacro (robot description, xacro)
@@ -65,4 +65,11 @@
 		<axis xyz="0 0 0"/>
 	</joint>
+	<link name="HokuyoLaser_frame"/>
+	<joint name="LaserSensor/Hokuyo_sensor_fixedjoint" type="fixed">
+		<parent link="Tibia"/>
+		<child link="HokuyoLaser_frame"/>
+		<origin rpy="-3.14159 0 0" xyz="0.2 0 -0.289"/>
+		<axis xyz="0 0 0"/>
+	</joint>
 	<link name="ImuTorsoAccelerometer_frame"/>
 	<joint name="Accelerometer_sensor_fixedjoint" type="fixed">
